File: Legacy/Amiga2000CPLDSlot/videoslotadapter.sch (KiCad schematic (older format))
At the start: 17 parts, among them J1 Raspberry_Pi_2_3, J2 Conn_01x06, U1 XC9572VQ44

Commit message: Add Amiga 2000 CPLD v2.1
Adds the Amiga 2000 CPLD v2.1 and moves older boards to legacy.
Parts:
- removed H3, H4, H5, H6: MountingHole, MountingHole:MountingHole_2.7mm_M2.5, symbol Mechanical:MountingHole
- removed J2: Conn_01x06, Connector_PinHeader_2.54mm:PinHeader_1x06_P2.54mm_Horizontal, symbol Connector_Generic:Conn_01x06
- removed R3: 100, Resistor_SMD:R_0603_1608Metric_Pad0.98x0.95mm_HandSolder, symbol Device:R
- removed R4: 56, Resistor_SMD:R_0603_1608Metric_Pad0.98x0.95mm_HandSolder, symbol Device:R
- added JButton1, JButton2, JButton3, JButton4, JButton5, JButton6: Conn_01x02, Connector_PinHeader_2.54mm:PinHeader_1x02_P2.54mm_Horizontal, symbol Connector_Generic:Conn_01x02
Connections:
- wire segments 126 -> 132
